File: HPF.sch (KiCad schematic (older format))
At the start: 174 parts, among them J1 CONN_COAXIAL, J2 Conn_01x12, J3 CONN_COAXIAL, J4 CONN_COAXIAL, J5 CONN_COAXIAL, Q2 zvp2106G, U1 AP1117-50, U2 PGA103+

Commit message: new gerber
Parts:
- Q2: footprint TO_SOT_Packages_SMD:SOT-23_Handsoldering -> TO_SOT_Packages_SMD:SOT-223-3Lead_TabPin2
Changed lines of the file:
@@
 F 0 "Q2" H 2750 10100 50  0000 L CNN
 F 1 "zvp2106G" H 2650 10200 50  0000 L CNN
-F 2 "TO_SOT_Packages_SMD:SOT-23_Handsoldering" H 3250 9975 50  0001 L CIN
+F 2 "TO_SOT_Packages_SMD:SOT-223-3Lead_TabPin2" H 3250 9975 50  0001 L CIN
 F 3 "" H 3000 10050 50  0001 L CNN
 	1    3000 10050

Commit message: upgrate to Kicad 5.0n, new up to date Gerber
Parts:
- C1, C100, C101, C102, C103, C104, C106, C107, C108, C109, C110, C111, C112, C113, C115, C116, C117, C118, C119, C120, C121, C122, C123, C124, C125, C126, C127, C128, C129, C130, C131, C132, C133, C134, C135, C136, C137, C139, C140, C143, C144, C145, C146, C147, C148, C149, C150, C151, C152, C153, C154, C155, C156, C157, C158, C159, C160, C161, C162, C163, C183, C2, C3, C4, C76, C77, C78, C79, C80, C81, C82, C83, C84, C85, C86, C87, C88, C90, C91, C92, C93, C94, C95, C96, C97, C98: symbol C -> HPF-rescue:C
- C10, C11, C12, C13, C14, C15, C16, C5, C6, C7, C8, C9: symbol C_Small -> HPF-rescue:C_Small
- D1, D2, D3, D4, D5: symbol D -> HPF-rescue:D
- J1, J3, J4, J5: symbol CONN_COAXIAL -> HPF-rescue:CONN_COAXIAL
- J2: symbol Conn_01x12 -> HPF-rescue:Conn_01x12
- L1, L10, L11, L12, L13, L14, L15, L16, L18, L19, L2, L20, L21, L22, L24, L25, L26, L27, L28, L29, L3, L30, L31, L32, L33, L4, L5, L6, L7, L8, L9: symbol L_Core_Ferrite_Small -> HPF-rescue:L_Core_Ferrite_Small
- L17, L23, L34, L35: symbol L_Small -> HPF-rescue:L_Small
- Q2: symbol IRF9540N-RESCUE-HPF -> HPF-rescue:IRF9540N-RESCUE-HPF
- R1, R10, R11, R12, R13, R2: symbol R -> HPF-rescue:R
- R3, R5: symbol R_Small -> HPF-rescue:R_Small
- RL1, RL16, RL17, RL18, RL19, RL2, RL20, RL21, RL22, RL23, RL24, RL25, RL26, RL27, RL28, RL29: symbol EE2-5NU -> ee2-5nu:EE2-5NU
- TP1, TP2, TP3, TP4: symbol TEST -> HPF-rescue:TEST
- U1: symbol AP1117-50 -> HPF-rescue:AP1117-50
- U2: symbol PGA103+ -> pga103+:PGA103+
Other:
- note added: "RX_Master_IN"
